File: PCB/control board/control board.kicad_sch (KiCad schematic)
At the start: 27 parts

Commit message: footprint pro tlačítka a schéma pro control boardu
Parts:
- C1, C2, C3, C4, C5, C6, C7, C8: renamed from C?; footprint (none) -> Capacitor_SMD:C_0805_2012Metric_Pad1.18x1.45mm_HandSolder
- J1, J2, J3: renamed from J?; footprint (none) -> Connector_PinSocket_2.54mm:PinSocket_1x05_P2.54mm_Vertical
- R1, R2, R3, R4, R5, R6, R7, R8: renamed from R?; footprint (none) -> Resistor_SMD:R_0805_2012Metric_Pad1.20x1.40mm_HandSolder
- SW1, SW2, SW3, SW4, SW5, SW6, SW7, SW8: renamed from SW?; footprint (none) -> TL3301SPF160QG:TL3301SPF160QG

Commit message: Led board + control board
Parts:
- removed C6: 100nF, Capacitor_SMD:C_0805_2012Metric_Pad1.18x1.45mm_HandSolder, symbol Device:C_Small
- removed J1, J2, J3: JST-XH 1x05, Connector_PinSocket_2.54mm:PinSocket_1x05_P2.54mm_Vertical, symbol Connector:Conn_01x05_Female
- removed R6: 10k, Resistor_SMD:R_0805_2012Metric_Pad1.20x1.40mm_HandSolder, symbol Device:R_Small
- removed SW6, SW7: SW_MEC_5E, TL3301SPF160QG:TL3301SPF160QG, symbol Switch:SW_MEC_5E
- added C10, C2, C5, C9: 100nF, Capacitor_SMD:C_0805_2012Metric_Pad1.18x1.45mm_HandSolder, symbol Device:C_Small
- added J1: BTN1, Connector_PinSocket_2.54mm:PinSocket_1x02_P2.54mm_Vertical, symbol Connector:Conn_01x02_Female
- added J2: BTN2, Connector_PinSocket_2.54mm:PinSocket_1x02_P2.54mm_Vertical, symbol Connector:Conn_01x02_Female
- added J3: BTN3, symbol Connector:Conn_01x02_Female
- added J4: Conn_02x05_Top_Bottom, Connector_PinSocket_2.54mm:PinSocket_2x05_P2.54mm_Vertical, symbol Connector_Generic:Conn_02x05_Top_Bottom
- added R10, R2, R5, R9: 10k, Resistor_SMD:R_0805_2012Metric_Pad1.20x1.40mm_HandSolder, symbol Device:R_Small
- added SW2, SW5: SW_MEC_5E, TL3301SPF160QG:TL3301SPF160QG, symbol Switch:SW_MEC_5E
- renumbered C7 to C11, C2 to C3, C3 to C4, C4 to C6, C5 to C7, R7 to R11, R2 to R3, R3 to R4, R4 to R6, R5 to R7, SW2 to SW3, SW3 to SW4, SW4 to SW6, SW5 to SW7
Connections:
- net +3.3V: now also R10.2, R2.2, R5.2, R9.2
- net BTN1: now also C9.1, J1.2 (Pin_2), R9.1; no longer C8.1, SW8.3 (K)
- net BTN2: now also C10.1, J2.2 (Pin_2), R10.1
- net BTN3: now also R11.1, J3.2 (Pin_2)
- net GND: now also C10.2, C2.2, C5.2, C9.2, J1.1 (Pin_1), J2.1 (Pin_1), J3.1 (Pin_1), SW2.2, SW5.2
- new net: R5.1, SW5.4 (A)
- new net: R2.1, SW2.4 (A)
- new net BACK: C8.1, SW8.3 (K)
- new net HOME: C5.1, SW5.3 (K)
- new net MENU: C2.1, SW2.3 (K)
- no-connect marks 13 -> 8
Other:
- note added: "IO expandér"
- note added: "Menu"
- note removed: "Konektory"
- note removed: "Neosazovat-rezerva navíc"
- moved on the sheet: C1, C11, C3, C4, C6, C7, R1, R11, R3, R4, R6, R7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

Commit message: control a led boarda hotový kromě popisku a děr
Parts:
- added C6: 100nF, Capacitor_SMD:C_0805_2012Metric_Pad1.18x1.45mm_HandSolder, symbol Device:C_Small
- added R4, R5, R6: 10k, Resistor_SMD:R_0805_2012Metric_Pad1.20x1.40mm_HandSolder, symbol Device:R_Small
- added U1: PCA9555D, Package_SO:SOIC-24W_7.5x15.4mm_P1.27mm, symbol Interface_Expansion:PCA9555D
- J3: renamed from J4; value Conn_02x05_Top_Bottom -> IDC_CONN
- renumbered C2 to C1, C7 to C10, C4 to C12, C5 to C2, C8 to C3, C9 to C4, C6 to C5, C10 to C7, C1 to C8, C3 to C9, J3 to J4, R2 to R1, R3 to R10, R7 to R11, R10 to R12, R4 to R13, R11 to R14, R5 to R2, R8 to R3, R6 to R7, R9 to R8, R1 to R9, SW2 to SW1, SW5 to SW2, SW8 to SW3, SW6 to SW4, SW1 to SW5, SW3 to SW6, SW4 to SW8
Connections:
- net +3.3V: now also J3.1 (Pin_1), C6.1, R4.2, R5.2, R6.2, U1.24 (VDD)
- net BACK: now also U1.5 (IO0_1)
- net BTN1: now also U1.20 (IO1_7)
- net BTN2: now also U1.19 (IO1_6)
- net BTN3: now also U1.18 (IO1_5)
- net DOWN: now also U1.13 (IO1_0)
- net GND: now also J3.5 (Pin_5), C6.2, U1.12 (VSS), U1.2 (A1), U1.21 (A0), U1.3 (A2)
- net HOME: now also U1.4 (IO0_0)
- net LEFT: now also U1.14 (IO1_1)
- net MENU: now also U1.6 (IO0_2)
- net OK: now also U1.15 (IO1_2)
- net RIGHT: now also U1.16 (IO1_3)
- net SCL: now also J3.4 (Pin_4), R4.1, U1.22 (SCL)
- net SDA: now also J3.3 (Pin_3), R5.1, U1.23 (SDA)
- net UP: now also U1.17 (IO1_4)
- net INT: now reaches J3.2 (Pin_2)
- net INT: now also R6.1, U1.1 (~{INT})
- no-connect marks 8 -> 18
Other:
- note added: "Vstup"
- moved on the sheet: J3
