File: PCB/LED board/LED board.kicad_pcb (KiCad board)
At the start: 2 copper layers, 99.3 x 84.6 mm, 9 parts, among them J1 Conn_01x14_Female, J2 Conn_02x05_IDC

Commit message: mount pro control,LED board.Komplet sensor board
Parts:
- added ?: , , F.Cu at (125.7, 129.0)
- added ?: , , F.Cu at (212.1, 145.8)
- added ?: , , F.Cu at (121.4, 71.1)
Routing:
- net GND: vias 0 -> 23
Other:
- outline, holes or cut-outs redrawn
- board text added: "GORAK INDUSTRIES Project FENIX LED board V1.0"
