File: PCB/LED board/LED board_V1.0.kicad_pcb (KiCad board)
At the start: 2 copper layers, 99.3 x 84.6 mm, 12 parts, among them J1 Conn_01x14_Female, J2 Conn_02x05_IDC

Commit message: uklizení souboru_V1.0
Other:
- board text added: "${REVISION}"
Changed lines of the file:
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@@
   (gr_circle (center 213.284 71.12) (end 214.884 71.12) (layer "Edge.Cuts") (width 0.1) (fill none))
   (gr_circle (center 213.284 121.158) (end 214.884 121.158) (layer "Edge.Cuts") (width 0.1) (fill none))
+  (gr_text "${REVISION}" (at 150.114 144.526) (layer "F.SilkS")
+    (effects (font (size 1 1) (thickness 0.15)))
+  )
   (gr_text "GORAK INDUSTRIES\nProject FENIX\nLED board V1.0" (at 192.532 145.034) (layer "F.SilkS")
     (effects (font (size 2 2) (thickness 0.15)))
   )
-  (dimension (type aligned) (layer "F.SilkS")
-    (pts (xy 216.154 65.532) (xy 117.094 65.532))
-    (height 2.794)
-    (gr_text "99,0600 mm" (at 166.624 61.588) (layer "F.SilkS")
-      (effects (font (size 1 1) (thickness 0.15)))
-    )
-    (format (units 3) (units_format 1) (precision 4))
-    (style (thickness 0.15) (arrow_length 1.27) (text_position_mode 0) (extension_height 0.58642) (extension_offset 0.5) keep_text_aligned)
+  (gr_text "${REVISION}" (at 149.86 145.542) (layer "F.SilkS")
+    (effects (font (size 1 1) (thickness 0.15)))
   )
-  (dimension (type aligned) (layer "F.SilkS")
-    (pts (xy 216.408 150.368) (xy 216.408 65.532))
-    (height 5.08)
-    (gr_text "84,8360 mm" (at 220.338 107.95 90) (layer "F.SilkS")
+  (dimension (type aligned) (layer "Dwgs.User")
+    (pts (xy 216.408 150.114) (xy 117.094 150.114))
+    (height -2.54)
+    (gr_text "99,3140 mm" (at 166.751 151.504) (layer "Dwgs.User")
       (effects (font (size 1 1) (thickness 0.15)))
     )
@@
   (dimension (type aligned) (layer "Dwgs.User")
     (pts (xy 216.408 65.532) (xy 216.408 150.114))
-    (height -4.826)
-    (gr_text "84,5820 mm" (at 220.084 107.823 90) (layer "Dwgs.User")
+    (height -3.556)
+    (gr_text "84,5820 mm" (at 218.814 107.823 90) (layer "Dwgs.User")
       (effects (font (size 1 1) (thickness 0.15)))
     )
-    (format (units 3) (units_format 1) (precision 4))
-    (style (thickness 0.15) (arrow_length 1.27) (text_position_mode 0) (extension_height 0.58642) (extension_offset 0.5) keep_text_aligned)
-  )
-  (dimension (type aligned) (layer "Dwgs.User")
-    (pts (xy 216.408 150.114) (xy 117.094 150.114))
-    (height -5.334)
-    (gr_text "99,3140 mm" (at 166.751 154.298) (layer "Dwgs.User")
-      (effects (font (size 1 1) (thickness 0.15)))
-    )
