File: PCB/Sensor/sensor board/sensor board.kicad_sch (KiCad schematic)
At the start: 24 parts, among them J1 Conn_01x07, J2 JST-XH, J3 INPUT, SW1 SW_Push, SW2 SW_Push, U1 ESP32-S3-WROOM-1-N16R2

Commit message: sensor V1.1 + gerbery
Parts:
- removed SW1, SW2: SW_Push, Button_Switch_SMD:SW_SPST_CK_RS282G05A3, symbol Switch:SW_Push
Changed lines of the file:
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@@
     (title "Sensor board")
     (date "2023-04-15")
-    (rev "V1.0")
+    (rev "V1.1")
     (company "GORAK INDUSTRIES")
   )
@@
   (junction (at 101.6 74.93) (diameter 0) (color 0 0 0 0)
   )
-  (junction (at 76.2 85.09) (diameter 0) (color 0 0 0 0)
-  )
   (junction (at 229.87 127) (diameter 0) (color 0 0 0 0)
   )
@@
   )
   (junction (at 165.1 114.3) (diameter 0) (color 0 0 0 0)
-  )
-  (junction (at 101.6 85.09) (diameter 0) (color 0 0 0 0)
   )
   (junction (at 68.58 107.95) (diameter 0) (color 0 0 0 0)
@@
     (stroke (width 0) (type default) (color 0 0 0 0))
   )
-  (wire (pts (xy 76.2 85.09) (xy 76.2 81.28))
+  (wire (pts (xy 76.2 81.28) (xy 76.2 86.36))
     (stroke (width 0) (type default) (color 0 0 0 0))
   )
@@
     (stroke (width 0) (type default) (color 0 0 0 0))
   )
-  (wire (pts (xy 66.04 85.09) (xy 76.2 85.09))
-    (stroke (width 0) (type default) (color 0 0 0 0))
-  )
   (wire (pts (xy 101.6 73.66) (xy 101.6 74.93))
     (stroke (width 0) (type default) (color 0 0 0 0))
@@
     (stroke (width 0) (type default) (color 0 0 0 0))
   )
-  (wire (pts (xy 66.04 74.93) (xy 76.2 74.93))
-    (stroke (width 0) (type default) (color 0 0 0 0))
-  )
   (wire (pts (xy 69.85 113.03) (xy 68.58 113.03))
     (stroke (width 0) (type default) (color 0 0 0 0))
@@
     (stroke (width 0) (type default) (color 0 0 0 0))
   )
-  (wire (pts (xy 76.2 86.36) (xy 76.2 85.09))
-    (stroke (width 0) (type default) (color 0 0 0 0))
-  )
   (wire (pts (xy 176.53 71.12) (xy 176.53 69.85))
     (stroke (width 0) (type default) (color 0 0 0 0))
@@
     (stroke (width 0) (type default) (color 0 0 0 0))
   )
-  (wire (pts (xy 91.44 85.09) (xy 101.6 85.09))
-    (stroke (width 0) (type default) (color 0 0 0 0))
-  )
   (polyline (pts (xy 114.3 96.52) (xy 114.3 132.08))
     (stroke (width 0) (type default) (color 0 0 0 0))
@@
     (stroke (width 0) (type default) (color 0 0 0 0))
   )
-  (wire (pts (xy 91.44 74.93) (xy 101.6 74.93))
-    (stroke (width 0) (type default) (color 0 0 0 0))
-  )
   (wire (pts (xy 165.1 106.68) (xy 168.91 106.68))
     (stroke (width 0) (type default) (color 0 0 0 0))
   )
-  (wire (pts (xy 101.6 85.09) (xy 101.6 81.28))
-    (stroke (width 0) (type default) (color 0 0 0 0))
-  )
   (wire (pts (xy 165.1 74.93) (xy 166.37 74.93))
     (stroke (width 0) (type default) (color 0 0 0 0))
@@
     (stroke (width 0) (type default) (color 0 0 0 0))
   )
-  (wire (pts (xy 101.6 86.36) (xy 101.6 85.09))
+  (wire (pts (xy 101.6 81.28) (xy 101.6 86.36))
     (stroke (width 0) (type default) (color 0 0 0 0))
   )
@@
     (pin "2")
   )
-  (symbol (lib_id "Switch:SW_Push") (at 91.44 80.01 90) (unit 1)
-    (in_bom yes) (on_board yes) (fields_autoplaced)
-    (property "Reference" "SW2" (id 0) (at 92.71 78.7399 90)
-      (effects (font (size 1.27 1.27)) (justify right))
-    )
-    (property "Value" "SW_Push" (id 1) (at 92.71 81.2799 90)
-      (effects (font (size 1.27 1.27)) (justify right))
-    )
-    (property "Footprint" "Button_Switch_SMD:SW_SPST_CK_RS282G05A3" (id 2) (at 86.36 80.01 0)
-      (effects (font (size 1.27 1.27)) hide)
-    )
-    (property "Datasheet" "~" (id 3) (at 86.36 80.01 0)
-      (effects (font (size 1.27 1.27)) hide)
-    )
-    (pin "1")
-    (pin "2")
-  )
   (symbol (lib_id "power:GND") (at 123.19 123.19 0) (unit 1)
     (in_bom yes) (on_board yes)
@@
     (pin "2")
   )
-  (symbol (lib_id "Switch:SW_Push") (at 66.04 80.01 90) (unit 1)
-    (in_bom yes) (on_board yes) (fields_autoplaced)
-    (property "Reference" "SW1" (id 0) (at 67.31 78.7399 90)
-      (effects (font (size 1.27 1.27)) (justify right))
-    )
-    (property "Value" "SW_Push" (id 1) (at 67.31 81.2799 90)
-      (effects (font (size 1.27 1.27)) (justify right))
-    )
-    (property "Footprint" "Button_Switch_SMD:SW_SPST_CK_RS282G05A3" (id 2) (at 60.96 80.01 0)
-      (effects (font (size 1.27 1.27)) hide)
-    )
-    (property "Datasheet" "~" (id 3) (at 60.96 80.01 0)
-      (effects (font (size 1.27 1.27)) hide)
-    )
-    (pin "1")
-    (pin "2")
-  )
   (symbol (lib_id "power:GND") (at 76.2 86.36 0) (unit 1)
     (in_bom yes) (on_board yes)
@@
       (reference "R9") (unit 1) (value "15k") (footprint "Resistor_SMD:R_0805_2012Metric_Pad1.20x1.40mm_HandSolder")
     )
-    (path "/d501c30b-9087-482c-b539-2eea225adb24"
-      (reference "SW1") (unit 1) (value "SW_Push") (footprint "Button_Switch_SMD:SW_SPST_CK_RS282G05A3")
-    )
-    (path "/96c31241-6aab-47f2-ad1e-559f03503a94"
-      (reference "SW2") (unit 1) (value "SW_Push") (footprint "Button_Switch_SMD:SW_SPST_CK_RS282G05A3")
-    )
     (path "/3fbdb62d-558d-49b5-a976-c70e20e6531f"
